File: PCB/Main/Main.kicad_pcb (KiCad board)
At the start: 2 copper layers, 6 parts, among them J1 Lidar1, J2 Lidar1, J3 Lidar1, J4 Lidar1, J5 Raspberry_Pi_2_3, U1 ESP32-DEVKITC

Commit message: commit
Parts:
- added H1: MountingHole_Pad, MountingHole:MountingHole_4mm_Pad_Via, F.Cu at (117.0, 69.5)
- added H2: MountingHole_Pad, MountingHole:MountingHole_4mm_Pad_Via, F.Cu at (165.0, 55.0)
- added H3: MountingHole_Pad, MountingHole:MountingHole_4mm_Pad_Via, F.Cu at (178.0, 110.0)
- added H4: MountingHole_Pad, MountingHole:MountingHole_4mm_Pad_Via, F.Cu at (189.9, 110.0)
- added H5: MountingHole_Pad, MountingHole:MountingHole_4mm_Pad_Via, F.Cu at (167.1, 110.0)
- added H6: MountingHole_Pad, MountingHole:MountingHole_4mm_Pad_Via, F.Cu at (153.9, 110.1)
- added J10: Conn_01x03, Connector_PinHeader_2.54mm:PinHeader_1x03_P2.54mm_Vertical, F.Cu at (55.0, 77.5)
- added J6: ToF1, Connector_PinSocket_2.54mm:PinSocket_1x06_P2.54mm_Horizontal, F.Cu at (78.7, 104.6)
- added J7: ToF2, Connector_PinSocket_2.54mm:PinSocket_1x06_P2.54mm_Horizontal, F.Cu at (185.0, 80.0)
- added J8: ToF3, Connector_PinSocket_2.54mm:PinSocket_1x06_P2.54mm_Horizontal, F.Cu at (91.3, 40.4)
- added J9: ToF4, Connector_PinSocket_2.54mm:PinSocket_1x06_P2.54mm_Horizontal, F.Cu at (50.0, 87.8)
- added M1: Motor_Servo, Connector_PinHeader_2.54mm:PinHeader_1x03_P2.54mm_Vertical, F.Cu at (123.0, 38.5)
- added PLogic1: ~, Connector_PinHeader_2.54mm:PinHeader_1x04_P2.54mm_Vertical, F.Cu at (182.0, 56.0)
- added PMotor1: ~, Connector_PinHeader_2.54mm:PinHeader_1x04_P2.54mm_Vertical, F.Cu at (182.2, 84.0)
- added TP1: TestPoint, Pegoku:TestPoint, F.Cu at (124.5, 72.5)
- added TP2: TestPoint, Pegoku:TestPoint, F.Cu at (161.5, 66.5)
- added U2: XT60, easyeda2kicad:CONN-TH_XT60, F.Cu at (143.0, 96.6)
- J1: footprint Connector_PinHeader_2.54mm:PinHeader_1x04_P2.54mm_Horizontal -> Connector_PinHeader_2.54mm:PinHeader_1x04_P2.54mm_Vertical
- J2: value Lidar1 -> Lidar2; footprint Connector_PinHeader_2.54mm:PinHeader_1x04_P2.54mm_Horizontal -> Connector_PinHeader_2.54mm:PinHeader_1x04_P2.54mm_Vertical
- J3: value Lidar1 -> Lidar3; footprint Connector_PinHeader_2.54mm:PinHeader_1x04_P2.54mm_Horizontal -> Connector_PinHeader_2.54mm:PinHeader_1x04_P2.54mm_Vertical
- J4: value Lidar1 -> Lidar4; footprint Connector_PinHeader_2.54mm:PinHeader_1x04_P2.54mm_Horizontal -> Connector_PinHeader_2.54mm:PinHeader_1x04_P2.54mm_Vertical
- J5: moved to F.Cu
- U1: value ESP32-DEVKITC -> L298N; footprint easyeda2kicad:BULETM-SMD_ESP32-DEVKITC -> Package_TO_SOT_THT:TO-220-15_P2.54x2.54mm_StaggerOdd_Lead4.58mm_Vertical
- moved J2 106.7 mm to (180.0, 69.2)
- moved J1 65.5 mm to (89.4, 101.0), turned to -90 degrees
- moved J4 31.5 mm to (55.0, 98.0), turned to 180 degrees
- moved J5 19.0 mm to (44.5, 34.1), turned to 0 degrees
- moved J3 17.7 mm to (81.4, 45.0), turned to 90 degrees
- moved U1 13.1 mm to (122.1, 61.4), turned to 90 degrees
Connections:
- net Net-(J5-3V3-Pad1) renamed +3.3V
- J1 pad 2: Net-(J1-Pin_2) -> unconnected-(J1-Pin_2-Pad2)
- J2 pad 1: Net-(J2-Pin_1) -> unconnected-(J2-Pin_1-Pad1)
- J3 pad 2: Net-(J3-Pin_2) -> unconnected-(J3-Pin_2-Pad2)
- J4 pad 2: Net-(J4-Pin_2) -> unconnected-(J4-Pin_2-Pad2)
- J5 pad 11: unconnected-(J5-GPIO17-Pad11) -> Net-(J5-GPIO17)
- J5 pad 14: Net-(J5-GND-Pad14) -> GND
- J5 pad 15: unconnected-(J5-GPIO22-Pad15) -> Net-(J1-Pin_1)
- J5 pad 16: unconnected-(J5-GPIO23-Pad16) -> Net-(J2-Pin_2)
- J5 pad 18: unconnected-(J5-GPIO24-Pad18) -> Net-(J3-Pin_1)
- J5 pad 19: unconnected-(J5-MOSI0/GPIO10-Pad19) -> Net-(J5-MOSI0/GPIO10)
- J5 pad 2: Net-(J5-5V-Pad2) -> +5V
- J5 pad 20: Net-(J5-GND-Pad14) -> GND
- J5 pad 22: unconnected-(J5-GPIO25-Pad22) -> Net-(J4-Pin_1)
- J5 pad 23: unconnected-(J5-SCLK0/GPIO11-Pad23) -> Net-(J5-SCLK0/GPIO11)
- J5 pad 25: Net-(J5-GND-Pad14) -> GND
- J5 pad 3: unconnected-(J5-SDA/GPIO2-Pad3) -> SDA
- J5 pad 30: Net-(J5-GND-Pad14) -> GND
- J5 pad 32: unconnected-(J5-PWM0/GPIO12-Pad32) -> Net-(J5-PWM0/GPIO12)
- J5 pad 34: Net-(J5-GND-Pad14) -> GND
- J5 pad 39: Net-(J5-GND-Pad14) -> GND
- J5 pad 4: Net-(J5-5V-Pad2) -> +5V
- J5 pad 5: unconnected-(J5-SCL/GPIO3-Pad5) -> SCL
- J5 pad 6: Net-(J5-GND-Pad14) -> GND
- J5 pad 9: Net-(J5-GND-Pad14) -> GND
- U1 pad 10: Net-(J3-Pin_1) -> unconnected-(U1-IN3-Pad10)
- U1 pad 11: Net-(J4-Pin_2) -> unconnected-(U1-EnB-Pad11)
- U1 pad 12: Net-(J4-Pin_1) -> unconnected-(U1-IN4-Pad12)
- U1 pad 14: GND -> unconnected-(U1-OUT4-Pad14)
- U1 pad 2: unconnected-(U1-EN-Pad2) -> Net-(U1-OUT1)
- U1 pad 3: unconnected-(U1-VP-Pad3) -> Net-(U1-OUT2)
- U1 pad 4: unconnected-(U1-VN-Pad4) -> VCCMotor
- U1 pad 5: Net-(J1-Pin_2) -> Net-(J5-MOSI0/GPIO10)
- U1 pad 6: Net-(J1-Pin_1) -> Net-(J5-PWM0/GPIO12)
- U1 pad 7: Net-(J2-Pin_2) -> Net-(J5-SCLK0/GPIO11)
- U1 pad 8: Net-(J2-Pin_1) -> GND
- U1 pad 9: Net-(J3-Pin_2) -> +5V
Routing:
- net GND: track 0.00 -> 407.0 mm, vias 0 -> 22
- net +5V: track 0.00 -> 288.4 mm, vias 0 -> 4
- net SDA: track 0.00 -> 259.7 mm, vias 0 -> 1
- net SCL: track 0.00 -> 246.5 mm, vias 0 -> 1
- net PowerToF: track 0.00 -> 243.8 mm, vias 0 -> 1
- net Net-(J2-Pin_2): track 0.00 -> 153.4 mm
- net +3.3V: track 0.00 -> 138.6 mm
- net VCCMotor: track 0.00 -> 136.9 mm, vias 0 -> 1
- net VCC: track 0.00 -> 110.2 mm
- net Net-(J5-GPIO17): track 0.00 -> 83.8 mm, vias 0 -> 1
- net Net-(J5-PWM0/GPIO12): track 0.00 -> 83.0 mm, vias 0 -> 1
- net Net-(J5-SCLK0/GPIO11): track 0.00 -> 81.0 mm
- net Net-(U1-OUT2): track 0.00 -> 79.7 mm
- net Net-(J5-MOSI0/GPIO10): track 0.00 -> 77.8 mm, vias 0 -> 1
- net Net-(J1-Pin_1): track 0.00 -> 70.6 mm
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- added copper zone on B.Cu, net GND
- added copper zone on F.Cu, net GND
Other:
- board outline added: 155 x 85 mm
- board text added: "3.3V"
- board text added: "5V"
- board text added: "EnA"
- board text added: "GND"
- board text added: "In1"
- board text added: "In2"
- board text added: "L298N"
- board text added: "Out 1"
- board text added: "Out 2"
- board text added: "Out1"
- board text added: "Out2"
- board text added: "PowerToF"
- board text added: "Servo"
- board text added: "ToF"
- board text added: "VCC In"
- board text added: "VCCMotor Out"
- board text added: "VCc(Vin) GND +5V GND"
- board text added: "Vcc"
