File: PCB/Main/Main.kicad_sch (KiCad schematic)
At the start: 9 parts, among them J1 Lidar1, J2 Lidar2, J3 Lidar3, J4 Lidar4, J5 Raspberry_Pi_2_3, J6 ToF1, J7 ToF2, J8 ToF3, J9 ToF4

Commit message: commit
Parts:
- added H1, H2, H3, H4, H5, H6: MountingHole_Pad, MountingHole:MountingHole_4mm_Pad_Via, symbol Mechanical:MountingHole_Pad
- added J10: Conn_01x03, Connector_PinHeader_2.54mm:PinHeader_1x03_P2.54mm_Vertical, symbol Connector_Generic:Conn_01x03
- added M1: Motor_Servo, Connector_PinHeader_2.54mm:PinHeader_1x03_P2.54mm_Vertical, symbol Motor:Motor_Servo
- added PLogic1, PMotor1: ~, Connector_PinHeader_2.54mm:PinHeader_1x04_P2.54mm_Vertical, symbol easyeda2kicad:AZXL4016E1
- added TP1, TP2: TestPoint, Pegoku:TestPoint, symbol Connector:TestPoint
- added U1: L298N, Package_TO_SOT_THT:TO-220-15_P2.54x2.54mm_StaggerOdd_Lead4.58mm_Vertical, symbol Driver_Motor:L298N
- added U2: XT60, easyeda2kicad:CONN-TH_XT60, symbol easyeda2kicad:XT60
- J1, J2, J3, J4: footprint Connector_PinHeader_2.54mm:PinHeader_1x04_P2.54mm_Horizontal -> Connector_PinHeader_2.54mm:PinHeader_1x04_P2.54mm_Vertical
Connections:
- net +3.3V: now also J10.3 (Pin_3), M1.2 (+); no longer J6.1 (Pin_1), J7.1 (Pin_1), J8.1 (Pin_1), J9.1 (Pin_1)
- net +5V: now also J10.1 (Pin_1), PLogic1.3 (Vout), U1.9 (Vss)
- net GND: now also J6.5 (Pin_5), J7.5 (Pin_5), J8.5 (Pin_5), J9.5 (Pin_5), H4.1, H6.1, M1.3 (-), PLogic1.2 (GND), PLogic1.4 (GND), PMotor1.2 (GND), PMotor1.4 (GND), U1.8 (GND), U2.1 (-); no longer J6.2 (Pin_2), J7.2 (Pin_2), J8.2 (Pin_2), J9.2 (Pin_2)
- net SCL: now also J6.4 (Pin_4), J7.4 (Pin_4), J8.4 (Pin_4), J9.4 (Pin_4); no longer J6.3 (Pin_3), J7.3 (Pin_3), J8.3 (Pin_3), J9.3 (Pin_3)
- net SDA: now also J6.3 (Pin_3), J7.3 (Pin_3), J8.3 (Pin_3), J9.3 (Pin_3); no longer J6.4 (Pin_4), J7.4 (Pin_4), J8.4 (Pin_4), J9.4 (Pin_4)
- net PowerToF: now reaches J8.6 (Pin_6)
- net PowerToF: now also J6.6 (Pin_6), J7.6 (Pin_6), J9.6 (Pin_6), J10.2 (Pin_2)
- net at J5.11 (GPIO17): now also M1.1 (PWM)
- net at J5.19 (MOSI0/GPIO10): now also U1.5 (IN1)
- net at J5.23 (SCLK0/GPIO11): now also U1.7 (IN2)
- net at J5.32 (PWM0/GPIO12): now also U1.6 (EnA)
- new net: H1.1, TP1.1, U1.2 (OUT1)
- new net: H2.1, TP2.1, U1.3 (OUT2)
- new net VCC: H5.1, PLogic1.1 (Vin), PMotor1.1 (Vin), U2.2 (+)
- new net VCCMotor: H3.1, PMotor1.3 (Vout), U1.4 (Vs)
